Commit message: urdf update

File: src/mobile_manipulator_body/urdf/mobile_manipulator.urdf (robot description, URDF)
Before this commit: robot mobile_manipulator, 10 links, 9 joints
Links:
- added link hand_link, mass 1.684558; collision mesh filename=package://mobile_manipulator_body/meshes/RG2_Hand_col.STL; visual mesh filename=package://mobile_manipulator_body/meshes/RG2_Hand_vis.STL
- added link l_finger_link, mass 0.081638; collision mesh filename=package://mobile_manipulator_body/meshes/RG2_LeftFinger_col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; visual mesh filename=package://mobile_manipulator_body/meshes/RG2_LeftFinger_vis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
- added link l_moment_arm_link, mass 0.160209; collision mesh filename=package://mobile_manipulator_body/meshes/RG2_LeftMomentArm_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; visual mesh filename=package://mobile_manipulator_body/meshes/RG2_LeftMomentArm_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
- added link l_truss_arm_link, mass 0.065927; collision mesh filename=package://mobile_manipulator_body/meshes/RG2_LeftTrussArm_c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; visual mesh filename=package://mobile_manipulator_body/meshes/RG2_LeftTrussArm_v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
Joints:
- added joint gripper_joint: type revolute, parent hand_link, child l_moment_arm_link, origin xyz=0.105 0.017 0.010 rpy=0 0 0, axis 0 0 1, limit lower=-0.45 upper=1.57 effort=10.6 velocity=3.14
- added joint hand_wrist_joint: type continuous, parent top_wrist, child hand_link, origin xyz=0.000 0.000 0.135 rpy=0 -1.57 0
- added joint l_finger_2_joint: type revolute, parent l_moment_arm_link, child l_finger_link, origin xyz=0.049 0.026 0.000 rpy=0 0 0, axis 0 0 1, limit lower=-1.57 upper=1.57 effort=10.6 velocity=3.14, mimic joint=gripper_joint multiplier=-1
- added joint l_finger_passive_joint: type revolute, parent hand_link, child l_truss_arm_link, origin xyz=0.122 0.008 0.010 rpy=0 0 0, axis 0 0 1, limit lower=-1.57 upper=1.57 effort=10.6 velocity=3.14, mimic joint=gripper_joint multiplier=1

Commit message: urdf update new

File: src/mobile_manipulator_body/urdf/mobile_manipulator.urdf (robot description, URDF)
Before this commit: robot mobile_manipulator, 14 links, 13 joints
Links:
- added link r_finger_link, mass 0.081637; collision mesh filename=package://mobile_manipulator_body/meshes/RG2_RightFinger_co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; visual mesh filename=package://mobile_manipulator_body/meshes/RG2_RightFinger_vi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
- added link r_moment_arm_link, mass 0.160209; collision mesh filename=package://mobile_manipulator_body/meshes/RG2_RightMomentArm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; visual mesh filename=package://mobile_manipulator_body/meshes/RG2_RightMomentArm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
- added link r_truss_arm_link, mass 0.065927; collision mesh filename=package://mobile_manipulator_body/meshes/RG2_RightTrussArm_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; visual mesh filename=package://mobile_manipulator_body/meshes/RG2_RightTrussArm_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
Joints:
- added joint r_finger_1_joint: type revolute, parent hand_link, child r_moment_arm_link, origin xyz=0.105 -0.017 0.010 rpy=0 0 0, axis 0 0 1, limit lower=-1.57 upper=1.57 effort=10.6 velocity=3.14, mimic joint=gripper_joint multiplier=-1
- added joint r_finger_2_joint: type revolute, parent r_moment_arm_link, child r_finger_link, origin xyz=0.049 -0.026 0.000 rpy=0 0 0, axis 0 0 1, limit lower=-1.57 upper=1.57 effort=10.6 velocity=3.14, mimic joint=gripper_joint multiplier=1
- added joint r_finger_passive_joint: type revolute, parent hand_link, child r_truss_arm_link, origin xyz=0.122 -0.008 0.010 rpy=0 0 0, axis 0 0 1, limit lower=-1.57 upper=1.57 effort=10.6 velocity=3.14, mimic joint=gripper_joint multiplier=-1
- joint hand_wrist_joint: type continuous -> fixed

Commit message: arm_control.yaml and mobile_manipulator.urdf updated

File: src/mobile_manipulator_body/urdf/mobile_manipulator.urdf (robot description, URDF)
Before this commit: robot mobile_manipulator, 17 links, 16 joints
Joints:
- joint gripper_joint: limit lower=-0.45 upper=1.57 effort=10.6 velocity=3.14 -> lower=-0.523 upper=0.523 effort=10.6 velocity=3.14
- joint l_finger_2_joint: limit lower=-1.57 upper=1.57 effort=10.6 velocity=3.14 -> lower=-0.523 upper=0.523 effort=10.6 velocity=3.14
- joint l_finger_passive_joint: limit lower=-1.57 upper=1.57 effort=10.6 velocity=3.14 -> lower=-0.523 upper=0.523 effort=10.6 velocity=3.14
- joint r_finger_1_joint: limit lower=-1.57 upper=1.57 effort=10.6 velocity=3.14 -> lower=-0.523 upper=0.523 effort=10.6 velocity=3.14
- joint r_finger_2_joint: limit lower=-1.57 upper=1.57 effort=10.6 velocity=3.14 -> lower=-0.523 upper=0.523 effort=10.6 velocity=3.14
- joint r_finger_passive_joint: limit lower=-1.57 upper=1.57 effort=10.6 velocity=3.14 -> lower=-0.523 upper=0.523 effort=10.6 velocity=3.14
