Commit message: map error fixed

File: src/mobile_manipulator_body/urdf/lidar.xacro (robot description, xacro)
@@ -10,5 +10,5 @@
     <mu2>0.2</mu2>
   </gazebo>
-  <link name="laz_base">
+  <!--<link name="laz_base">
     <visual>
       <geometry>
@@ -25,5 +25,5 @@
       <inertia ixx="${(1/12) * 0.1 * (3 * base_radius * base_radius + base_height * base_height)}" ixy="0" ixz="0" iyy="${(1/12) * 0.1 * (3 * base_radius * base_radius + base_height * base_height)}" iyz="0" izz="${(1/2) * 0.1 * base_radius * base_radius}"/>
     </inertial>
-  </link>
+  </link>-->
   <link name="laz_rot">
     <visual>
@@ -78,10 +78,3 @@
    </sensor>
   </gazebo>
-  <joint name="lazRot" type="revolute">
-    <parent link="laz_base"/>
-    <child link="laz_rot"/>
-    <axis xyz="0 0 1" rpy="0 0 0"/>
-    <limit effort="1000.0" lower="0.0" upper="0.0" velocity="0.0000001"/>
-    <origin xyz = "0 0 ${base_height/2}"/>
-  </joint>
 </robot>

File: src/mobile_manipulator_body/urdf/mobile_manipulator_gripper.urdf.xacro (robot description, xacro)
@@ -192,6 +192,6 @@
  <joint name="lidarGlue" type="fixed">
     <parent link="base_link"/>
-    <child link="laz_base"/>
-    <origin xyz="0.325 0 0" rpy = "0 ${pi/2} 0"/>
+    <child link="laz_rot"/>
+    <origin xyz="0.3 0.0 0.2" rpy = "0 0 0"/>
   </joint>
 <joint name="front_left_wheel_joint" type="continuous">
